File: Test PCB Designs/footprint_test/2018-Jan-Footprint-Test.kicad_pcb (KiCad board)
At the start: 2 copper layers, 25.4 x 38.1 mm, 4 parts, among them J1 Conn_01x05

Commit message: catchup
Parts:
- removed REF** (x2): MountingHole_3.2mm_M3, Mounting_Holes:MountingHole_3.2mm_M3
- J1: moved to B.Cu
- moved J1 17.3 mm to (128.1, 126.5), turned to 270 degrees
Routing:
- net Net-(J1-Pad4): track 30.0 -> 13.1 mm
- net Net-(J1-Pad2): track 35.0 -> 22.1 mm, vias 1 -> 0
- net Net-(J1-Pad3): track 23.3 -> 11.9 mm, vias 0 -> 1
- net Net-(J1-Pad5): track 7.33 -> 17.6 mm
Other:
- board outline removed
- board text added: "Joy v1.1"
- board text removed: "Xbox Joystick Footprint Test v1"
