File: Test PCB Designs/footprint_test/2018-Jan-Footprint-Test.sch (KiCad schematic (older format))
At the start: 2 parts, among them J1 Conn_01x05

Commit message: catchup
Parts:
- J1: symbol Conn_01x05 -> Connector_Generic:Conn_01x05
- JOY1: symbol xbox_joystick -> switches_inputs:xbox_joystick
Changed lines of the file:
@@
-EESchema Schematic File Version 2
-LIBS:power
-LIBS:device
-LIBS:switches
-LIBS:relays
-LIBS:motors
-LIBS:transistors
-LIBS:conn
-LIBS:linear
-LIBS:regul
-LIBS:74xx
-LIBS:cmos4000
-LIBS:adc-dac
-LIBS:memory
-LIBS:xilinx
-LIBS:microcontrollers
-LIBS:dsp
-LIBS:microchip
-LIBS:analog_switches
-LIBS:motorola
-LIBS:texas
-LIBS:intel
-LIBS:audio
-LIBS:interface
-LIBS:digital-audio
-LIBS:philips
-LIBS:display
-LIBS:cypress
-LIBS:siliconi
-LIBS:opto
-LIBS:atmel
-LIBS:contrib
-LIBS:valves
-LIBS:switches_inputs
+EESchema Schematic File Version 4
 LIBS:2018-Jan-Footprint-Test-cache
-EELAYER 25 0
+EELAYER 26 0
 EELAYER END
 $Descr A4 11693 8268
@@
 $EndDescr
 $Comp
-L xbox_joystick JOY1
+L switches_inputs:xbox_joystick JOY1
 U 1 1 5AA04B48
 P 1950 2300
@@
 $EndComp
 $Comp
-L Conn_01x05 J1
+L Connector_Generic:Conn_01x05 J1
 U 1 1 5AA04B7C
 P 2750 2300
@@
 	2150 2000 2150 2100
 Wire Wire Line
-	2150 2100 2550 2100
+	2150 2100 2350 2100
 Wire Wire Line
 	2150 2400 2350 2400
 Wire Wire Line
-	2350 2100 2350 2700
+	2350 2100 2350 2400
 Connection ~ 2350 2100
 Wire Wire Line
@@
 	2150 2300 2250 2300
 Wire Wire Line
-	2250 2200 2250 2600
+	2250 2200 2250 2300
 Wire Wire Line
 	2250 2200 2550 2200
@@
 Wire Wire Line
 	2500 2800 2150 2800
+Wire Wire Line
+	2350 2100 2550 2100
+Wire Wire Line
+	2350 2400 2350 2700
+Wire Wire Line
+	2250 2300 2250 2600
 $EndSCHEMATC
