File: Test PCB Designs/2020 05 PSP Joystick Breakout/2020 05 PSP Joystick Breakout.kicad_pcb (KiCad board)
At the start: 2 copper layers, 50.8 x 25.4 mm, 6 parts, among them J1 Conn_01x06, J2 SW1, J3 SW2

Commit message: PSP joystick prototype order
Parts:
- added G***: LOGO, BVH_Logos:SkyIron_logo_Back, F.Cu at (146.6, 126.0)
Changed lines of the file:
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@@
     (tracks 35)
     (zones 0)
-    (modules 6)
+    (modules 7)
     (nets 7)
   )
@@
       (outputformat 1)
       (mirror false)
-      (drillshape 1)
+      (drillshape 0)
       (scaleselection 1)
-      (outputdirectory ""))
+      (outputdirectory "order-2020-05-17/"))
   )
   (net 0 "")
@@
     (add_net Y)
   )
+  (module BVH_Logos:SkyIron_logo_Back (layer F.Cu)
+    (at 146.558 125.984)
+    (fp_text reference G*** (at 0 0) (layer F.SilkS) hide
+      (effects (font (size 1.524 1.524) (thickness 0.3)))
+    )
+    (fp_text value LOGO (at 0.75 0) (layer F.SilkS) hide
+      (effects (font (size 1.524 1.524) (thickness 0.3)))
+    )
+    (fp_poly (pts (xy 0.352298 -4.573742) (xy 0.020909 -4.517714) (xy -0.158124 -4.462771) (xy -0.568729 -4.218391)
+      (xy -0.960714 -3.860141) (xy -1.282732 -3.44029) (xy -1.423622 -3.174524) (xy -1.623737 -2.712223)
+      (xy -2.089404 -2.710306) (xy -2.720813 -2.641024) (xy -3.283692 -2.447098) (xy -3.754039 -2.141285)
+      (xy -4.107855 -1.736342) (xy -4.189405 -1.594084) (xy -4.327557 -1.193063) (xy -4.393634 -0.714943)
+      (xy -4.38447 -0.230464) (xy -4.296899 0.189635) (xy -4.272125 0.254) (xy -3.96779 0.76751)
+      (xy -3.543426 1.170759) (xy -3.017406 1.45105) (xy -2.408103 1.595686) (xy -2.318135 1.604313)
+      (xy -1.730121 1.651) (xy -2.206096 2.258653) (xy -2.415447 2.530443) (xy -2.57786 2.749903)
+      (xy -2.669836 2.884854) (xy -2.68207 2.910395) (xy -2.605941 2.940286) (xy -2.41146 2.9681)
+      (xy -2.262451 2.980076) (xy -1.842832 3.005667) (xy -2.43912 3.795609) (xy -2.66994 4.106555)
+      (xy -2.854143 4.364629) (xy -2.972683 4.542435) (xy -3.006906 4.612312) (xy -2.931538 4.575026)
+      (xy -2.734381 4.456125) (xy -2.434629 4.267785) (xy -2.051479 4.022182) (xy -1.604125 3.731492)
+      (xy -1.200404 3.46641) (xy 0.577596 2.293746) (xy -0.122819 2.268707) (xy -0.823235 2.243667)
+      (xy -0.299075 1.608667) (xy 1.917261 1.606807) (xy 2.5952 1.605383) (xy 3.126469 1.601369)
+      (xy 3.533727 1.593245) (xy 3.839631 1.579491) (xy 4.066842 1.558584) (xy 4.238018 1.529005)
+      (xy 4.375819 1.489233) (xy 4.502904 1.437746) (xy 4.514596 1.432483) (xy 5.028188 1.116403)
+      (xy 5.409697 0.701144) (xy 5.651277 0.20259) (xy 5.745077 -0.363375) (xy 5.700865 -0.836434)
+      (xy 3.502838 -0.836434) (xy 3.352551 -0.647268) (xy 3.106614 -0.344738) (xy 2.863604 -0.057756)
+      (xy 2.648923 0.184998) (xy 2.487973 0.354841) (xy 2.406159 0.423095) (xy 2.404315 0.423334)
+      (xy 2.319153 0.372883) (xy 2.140171 0.239209) (xy 1.902512 0.048824) (xy 1.846068 0.00215)
+      (xy 1.601324 -0.197243) (xy 1.408953 -0.346257) (xy 1.303542 -0.418301) (xy 1.295421 -0.421183)
+      (xy 1.230775 -0.358752) (xy 1.081728 -0.185219) (xy 0.867281 0.07642) (xy 0.606438 0.403172)
+      (xy 0.457611 0.592667) (xy -0.336024 1.608667) (xy -1.014169 1.608667) (xy -1.347314 1.606201)
+      (xy -1.538528 1.593901) (xy -1.615196 1.564409) (xy -1.604702 1.51037) (xy -1.565741 1.4605)
+      (xy -1.399739 1.259055) (xy -1.176672 0.978433) (xy -0.915862 0.644065) (xy -0.636634 0.281383)
+      (xy -0.35831 -0.084183) (xy -0.100215 -0.427202) (xy 0.118329 -0.722242) (xy 0.277996 -0.943873)
+      (xy 0.359465 -1.066663) (xy 0.36593 -1.081696) (xy 0.301878 -1.158891) (xy 0.129362 -1.309563)
+      (xy -0.122157 -1.508952) (xy -0.311404 -1.651) (xy -0.59765 -1.866231) (xy -0.824037 -2.045344)
+      (xy -0.961251 -2.164631) (xy -0.988737 -2.1988) (xy -0.913374 -2.243222) (xy -0.708531 -2.326799)
+      (xy -0.406075 -2.437298) (xy -0.06203 -2.554522) (xy 0.864676 -2.860681) (xy 2.183757 -1.848558)
+      (xy 3.502838 -0.836434) (xy 5.700865 -0.836434) (xy 5.69049 -0.94744) (xy 5.604056 -1.246889)
+      (xy 5.464262 -1.492027) (xy 5.229643 -1.753243) (xy 5.196794 -1.785465) (xy 4.811365 -2.090263)
+      (xy 4.38453 -2.276987) (xy 3.872369 -2.361616) (xy 3.588104 -2.370666) (xy 3.29564 -2.390779)
+      (xy 3.166767 -2.451268) (xy 3.159863 -2.4765) (xy 3.113249 -2.665778) (xy 2.990991 -2.943484)
+      (xy 2.819216 -3.262706) (xy 2.624052 -3.576536) (xy 2.431628 -3.838063) (xy 2.351763 -3.92734)
+      (xy 1.886228 -4.298801) (xy 1.359586 -4.518799) (xy 0.751632 -4.595544) (xy 0.706572 -4.595766)
+      (xy 0.352298 -4.573742)) (layer B.SilkS) (width 0.01))
+  )
   (module BVH_Components_Misc:PSP_Joystick_Hybrid (layer F.Cu)
