File: Test PCB Designs/2020 05 PSP Joystick Breakout/2020 05 PSP Joystick Breakout.sch (KiCad schematic (older format))
At the start: 4 parts, among them J1 Conn_01x06, J2 SW1, J3 SW2

Commit message: FPC Breakout Work
Parts:
- JOY1: symbol BVH_Sensors:PSP_Joystick -> 2020-05-PSP-Joystick-Breakout-rescue:PSP_Joystick-BVH_Sensors
Changed lines of the file:
@@
 SW2
 $Comp
-L BVH_Sensors:PSP_Joystick JOY1
+L 2020-05-PSP-Joystick-Breakout-rescue:PSP_Joystick-BVH_Sensors JOY1
 U 1 1 5EBEFAD9
 P 4900 2450
